File: CDEM.kicad_pcb (KiCad board)
At the start: 2 copper layers, 80.7 x 51.5 mm, 37 parts, among them J1 USB_C_Receptacle_USB2.0, J2 6P6C, Q1 2N7002, Q2 S8050, Q3 S8050, SW1 BTN, SW2 RESET, U1 AMS1117-3.3, U2 USBLC6-2SC6, U3 CP2104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

Commit message: finisching up the board
Parts:
- added J3: Conn_01x04, Connector_PinHeader_2.54mm:PinHeader_1x04_P2.54mm_Vertical, F.Cu at (71.3, 117.4)
- added L1: logo-devbit, cdem:logo_devbit_8mm, F.Cu at (47.4, 125.0)
- added L2: logo-vives, cdem:logo_vives_10mm, F.Cu at (79.5, 87.0)
- added REF**: OSHW-Logo2_9.8x8mm_SilkScreen, Symbol:OSHW-Logo2_9.8x8mm_SilkScreen, F.Cu at (84.4, 124.7)
Routing:
- net /USB-TX: track 37.6 -> 65.4 mm, vias 0 -> 2
- net /USB-RX: track 39.0 -> 66.2 mm
- net +3V3: track 89.2 -> 114.8 mm, vias 5 -> 7
- net GND: vias 97 -> 95
Other:
- board text added: "+3V3"
- board text added: "BOOT"
- board text added: "CDEM"
- board text added: "COMM"
- board text added: "DATA"
- board text added: "ESP-12E"
- board text added: "GND"
- board text added: "POWER"
- board text added: "RESET"
- board text added: "RX"
- board text added: "Sille Van Landschoot Nico De Witte Ronny Mees"
- board text added: "TX"

Commit message: add v4.0 laber on pcb
Other:
- board text added: "v4.0"
Changed lines of the file:
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@@
+    (effects (font (size 1 1) (thickness 0.15)))
+  )
+  (gr_text "v4.0" (at 41.6 94.8) (layer "F.SilkS")
     (effects (font (size 1 1) (thickness 0.15)))
   )

Commit message: final version v4.0
Parts:
- added R13: 1M, Resistor_SMD:R_0603_1608Metric, F.Cu at (55.6, 97.6)
Connections:
- net no_connect_58 renamed no_connect_56
- U3 pad 19: Net-(U3-Pad19) -> /RTS
- U3 pad 23: Net-(U3-Pad23) -> /DTR
Routing:
- net /RTS: track 2.15 -> 14.7 mm, vias 0 -> 2
- net /SM-DATA: track 48.7 -> 57.7 mm
- net /DTR: track 1.55 -> 6.56 mm
- net +3V3: track 114.8 -> 118.4 mm
- net /RESET: track 67.6 -> 64.6 mm, vias 0 -> 2
- net /GPIO0: track 54.7 -> 57.1 mm
- net Net-(R3-Pad2): track 60.2 -> 61.7 mm, vias 0 -> 2
- net GND: track 34.9 -> 35.9 mm
- net /USB-RX: track 66.2 -> 67.0 mm
- net /USB-TX: track 65.4 -> 66.2 mm

Commit message: fix power problem
Parts:
- removed D2: 1N4148W, Diode_SMD:D_SOD-123
- D1: value 1N4148W -> BAT54C; footprint Diode_SMD:D_SOD-123 -> Package_TO_SOT_SMD:SOT-23
- U1: value AMS1117-3.3 -> MCP1700-3302E_SOT23; footprint Package_TO_SOT_SMD:SOT-223-3_TabPin2 -> Package_TO_SOT_SMD:SOT-23
- moved U1 5.37 mm to (48.4, 107.4), turned to -90 degrees
- moved C3 3.25 mm to (48.4, 104.6), turned to 0 degrees
- moved D1 1.50 mm to (48.4, 111.0), turned to 90 degrees
- moved C1 0.53 mm to (51.3, 107.4), turned to 90 degrees
- moved Q2 0.10 mm to (62.0, 102.9)
Connections:
- D1 pad 1: Net-(C1-Pad1) -> VCC
- J1 pad A5: Net-(J1-PadA5) -> unconnected-(J1-PadA5)
- J1 pad A8: Net-(J1-PadA8) -> unconnected-(J1-PadA8)
- J1 pad B5: Net-(J1-PadB5) -> unconnected-(J1-PadB5)
- J1 pad B8: Net-(J1-PadB8) -> unconnected-(J1-PadB8)
- J2 pad 4: Net-(J2-Pad4) -> unconnected-(J2-Pad4)
- U3 pad 1: Net-(U3-Pad1) -> unconnected-(U3-Pad1)
- U3 pad 10: no_connect_56 -> unconnected-(U3-Pad10)
- U3 pad 11: Net-(U3-Pad11) -> unconnected-(U3-Pad11)
- U3 pad 12: Net-(U3-Pad12) -> unconnected-(U3-Pad12)
- U3 pad 13: Net-(U3-Pad13) -> unconnected-(U3-Pad13)
- U3 pad 14: Net-(U3-Pad14) -> unconnected-(U3-Pad14)
- U3 pad 15: Net-(U3-Pad15) -> unconnected-(U3-Pad15)
- U3 pad 17: Net-(U3-Pad17) -> unconnected-(U3-Pad17)
- U3 pad 18: Net-(U3-Pad18) -> unconnected-(U3-Pad18)
- U3 pad 22: Net-(U3-Pad22) -> unconnected-(U3-Pad22)
- U3 pad 24: Net-(U3-Pad24) -> unconnected-(U3-Pad24)
- U3 pad 9: Net-(U3-Pad9) -> unconnected-(U3-Pad9)
- U4 pad 10: Net-(U4-Pad10) -> unconnected-(U4-Pad10)
- U4 pad 11: Net-(U4-Pad11) -> unconnected-(U4-Pad11)
- U4 pad 12: Net-(U4-Pad12) -> unconnected-(U4-Pad12)
- U4 pad 13: Net-(U4-Pad13) -> unconnected-(U4-Pad13)
- U4 pad 14: Net-(U4-Pad14) -> unconnected-(U4-Pad14)
- U4 pad 19: Net-(U4-Pad19) -> unconnected-(U4-Pad19)
- U4 pad 2: Net-(U4-Pad2) -> unconnected-(U4-Pad2)
- U4 pad 4: Net-(U4-Pad4) -> unconnected-(U4-Pad4)
- U4 pad 9: Net-(U4-Pad9) -> unconnected-(U4-Pad9)
Routing:
- net GND: track 35.9 -> 21.8 mm
- net +3V3: track 118.4 -> 107.4 mm
- net Net-(C1-Pad1): track 7.94 -> 4.52 mm
- net /USB-IN-D-: track 17.7 -> 20.6 mm
- net VCC: track 49.2 -> 51.4 mm
- net VBUS: track 57.5 -> 55.7 mm
